File: pcb/rp3a0-mini-hdmi.kicad_sch (KiCad schematic)
At the start: 21 parts, among them J2 467652301, J3 1054500101, J4 SOLDER_PAD_OPEN, U1 RP3A0-AU, U5 DMN2004VK-7

Commit message: fix(pcb): resolve S2/S6/S7 validation findings across BOM, footprints, and 6-layer PCB
- Swap D1 (KT-0603G, C12624) symbol and PCB pad polarity so Pin 1 (K) connects to STATUS_LED and Pin 2 (A) to 3V3 via R11
- Replace U2 adjustable LCSC code with fixed 1.25V 500mA VBIAS LDO NCP133AMX125TCG (C603545) matching pinout and footprint
- Upgrade Y1 (S3219200182080C3, C5380596), U5 (DMN601VK-7, C110498), and R12/R13/R18 (RC0402FR-07240RL, C114755) to stocked JLCPCB parts
- Expand C0805_NP (C12, C14) inner pad gap to 0.70 mm and set 0 mm solder mask margin on fine-pitch U3 and J2
- Add D2 cathode bar, F.Fab/F.CrtYd outlines across all footprints, 3 global optical fiducials (FID1-FID3), and In4.Cu GND reference pour

Co-Authored-By: CopperPilot <noreply@copperpilot.ai>
Parts:
- U5: value DMN2004VK-7 -> DMN601VK-7; LCSC C145115 -> C110498; MPN DMN2004VK-7 -> DMN601VK-7
Changed lines of the file:
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@@
 			)
 		)
-		(property "Value" "DMN2004VK-7"
+		(property "Value" "DMN601VK-7"
 			(at 172.72 78.74 90)
 			(show_name no)
@@
 			)
 		)
-		(property "MPN" "DMN2004VK-7"
+		(property "MPN" "DMN601VK-7"
 			(at 180.34 66.04 0)
 			(effects
@@
 			)
 		)
-		(property "LCSC" "C145115"
+		(property "LCSC" "C110498"
 			(at 180.34 66.04 0)
 			(effects
