File: pcb/rp3a0-mini-misc.kicad_sch (KiCad schematic)
At the start: 16 parts, among them U1 RP3A0-AU

Commit message: fix(pcb): resolve S2/S6/S7 validation findings across BOM, footprints, and 6-layer PCB
- Swap D1 (KT-0603G, C12624) symbol and PCB pad polarity so Pin 1 (K) connects to STATUS_LED and Pin 2 (A) to 3V3 via R11
- Replace U2 adjustable LCSC code with fixed 1.25V 500mA VBIAS LDO NCP133AMX125TCG (C603545) matching pinout and footprint
- Upgrade Y1 (S3219200182080C3, C5380596), U5 (DMN601VK-7, C110498), and R12/R13/R18 (RC0402FR-07240RL, C114755) to stocked JLCPCB parts
- Expand C0805_NP (C12, C14) inner pad gap to 0.70 mm and set 0 mm solder mask margin on fine-pitch U3 and J2
- Add D2 cathode bar, F.Fab/F.CrtYd outlines across all footprints, 3 global optical fiducials (FID1-FID3), and In4.Cu GND reference pour

Co-Authored-By: CopperPilot <noreply@copperpilot.ai>
Parts:
- D1: LCSC C72043 -> C12624; MPN 19-217/GHC-YR1S2/3T -> KT-0603G
- R12, R13, R18: LCSC C25094 -> C114755; MPN 0402WGF2400TCE -> RC0402FR-07240RL
Connections:
- net at R11.2: now also D1.2; no longer D1.1
- net at U1.D4 (STATUS_LED): now also D1.1; no longer D1.2
Changed lines of the file:
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@@
 			)
 		)
-		(property "MPN" "0402WGF2400TCE"
+		(property "MPN" "RC0402FR-07240RL"
 			(at 149.86 76.2 0)
 			(effects
@@
 			)
 		)
-		(property "LCSC" "C25094"
+		(property "LCSC" "C114755"
 			(at 149.86 76.2 0)
 			(effects
@@
 			)
 		)
-		(property "MPN" "0402WGF2400TCE"
+		(property "MPN" "RC0402FR-07240RL"
 			(at 160.02 71.12 0)
 			(effects
@@
 			)
 		)
-		(property "LCSC" "C25094"
+		(property "LCSC" "C114755"
 			(at 160.02 71.12 0)
 			(effects
@@
 			)
 		)
-		(property "MPN" "0402WGF2400TCE"
+		(property "MPN" "RC0402FR-07240RL"
 			(at 154.94 68.58 0)
 			(effects
@@
 			)
 		)
-		(property "LCSC" "C25094"
+		(property "LCSC" "C114755"
 			(at 154.94 68.58 0)
 			(effects
@@
 			)
 		)
-		(property "Datasheet" "https://www.lcsc.com/product-detail/C72043.html"
+		(property "Datasheet" "https://www.lcsc.com/datasheet/lcsc_datasheet_1806151818_Hubei-KENTO-Elec-KT-0603G_C12624.pdf"
 			(at 81.28 83.82 0)
 			(hide yes)
@@
 			)
 		)
-		(property "MPN" "19-217/GHC-YR1S2/3T"
+		(property "MPN" "KT-0603G"
 			(at 81.28 83.82 0)
 			(effects
@@
 			)
 		)
-		(property "LCSC" "C72043"
+		(property "LCSC" "C12624"
 			(at 81.28 83.82 0)
 			(effects
