File: pcb/rp3a-mini-power.kicad_sch (KiCad schematic)
At the start: 67 parts, among them Q1 DMG2305UX-7, U1 RP3A0-AU, U2 RT9081A-1BGQZA(2), U3 RT8088AWSC, U4 PAM2306AYPKE, Y1 19.2MHz

Commit message: fix(pcb): update 19.2MHz crystal load caps to 27pF, add PCB title block, and export JLCPCB BOM/CPL
Update C6 and C9 from 18pF to 27pF (0402CG270J500NT, LCSC C1557) to provide 18.0 pF effective load capacitance for Y1 (ECS-192-18-33-JGN-TR), add PCB title_block metadata, and configure export_manufacturing.py with JLCPCB_CORRECTIONS and tracked pcb/jlcpcb/ BOM/CPL outputs.

Co-Authored-By: CopperPilot <noreply@copperpilot.ai>
Parts:
- C6, C9: value 18p -> 27p; LCSC C1549 -> C1557; MPN 0402CG180J500NT -> 0402CG270J500NT
Changed lines of the file:
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@@
 			)
 		)
-		(property "Value" "18p"
+		(property "Value" "27p"
 			(at 109.22 155.956 90)
 			(hide yes)
@@
 			)
 		)
-		(property "MPN" "0402CG180J500NT"
+		(property "MPN" "0402CG270J500NT"
 			(at 109.22 149.86 0)
 			(effects
@@
 			)
 		)
-		(property "LCSC" "C1549"
+		(property "LCSC" "C1557"
 			(at 109.22 149.86 0)
 			(effects
@@
 			)
 		)
-		(property "Value" "18p"
+		(property "Value" "27p"
 			(at 109.22 176.276 90)
 			(hide yes)
@@
 			)
 		)
-		(property "MPN" "0402CG180J500NT"
+		(property "MPN" "0402CG270J500NT"
 			(at 109.22 170.18 0)
 			(effects
@@
 			)
 		)
-		(property "LCSC" "C1549"
+		(property "LCSC" "C1557"
 			(at 109.22 170.18 0)
 			(effects

Commit message: fix(pcb): resolve S2/S6/S7 validation findings across BOM, footprints, and 6-layer PCB
- Swap D1 (KT-0603G, C12624) symbol and PCB pad polarity so Pin 1 (K) connects to STATUS_LED and Pin 2 (A) to 3V3 via R11
- Replace U2 adjustable LCSC code with fixed 1.25V 500mA VBIAS LDO NCP133AMX125TCG (C603545) matching pinout and footprint
- Upgrade Y1 (S3219200182080C3, C5380596), U5 (DMN601VK-7, C110498), and R12/R13/R18 (RC0402FR-07240RL, C114755) to stocked JLCPCB parts
- Expand C0805_NP (C12, C14) inner pad gap to 0.70 mm and set 0 mm solder mask margin on fine-pitch U3 and J2
- Add D2 cathode bar, F.Fab/F.CrtYd outlines across all footprints, 3 global optical fiducials (FID1-FID3), and In4.Cu GND reference pour

Co-Authored-By: CopperPilot <noreply@copperpilot.ai>
Parts:
- U2: value RT9081A-1BGQZA(2) -> NCP133AMX125TCG; LCSC C7303451 -> C603545; MPN RT9081A-1BGQZA(2) -> NCP133AMX125TCG
- Y1: LCSC C2450083 -> C5380596; MP ECS-192-18-33-JGN-TR -> S3219200182080C3; MPN ECS-192-18-33-JGN-TR -> S3219200182080C3
Changed lines of the file:
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@@
 			)
 		)
-		(property "MP" "ECS-192-18-33-JGN-TR"
+		(property "MP" "S3219200182080C3"
 			(at 114.3 160.02 90)
 			(hide yes)
@@
 			)
 		)
-		(property "MPN" "ECS-192-18-33-JGN-TR"
+		(property "MPN" "S3219200182080C3"
 			(at 114.3 160.02 0)
 			(effects
@@
 			)
 		)
-		(property "LCSC" "C2450083"
+		(property "LCSC" "C5380596"
 			(at 114.3 160.02 0)
 			(effects
@@
 			)
 		)
-		(property "Value" "RT9081A-1BGQZA(2)"
+		(property "Value" "NCP133AMX125TCG"
 			(at 170.18 71.12 90)
 			(show_name no)
@@
 			)
 		)
-		(property "Datasheet" "https://www.richtek.com/assets/product_file/RT9081A/DS9081A-05.pdf"
+		(property "Datasheet" "https://www.onsemi.com/download/data-sheet/pdf/ncp133-d.pdf"
 			(at 180.34 58.42 0)
 			(hide yes)
@@
 			)
 		)
-		(property "MPN" "RT9081A-1BGQZA(2)"
+		(property "MPN" "NCP133AMX125TCG"
 			(at 180.34 58.42 0)
 			(effects
@@
 			)
 		)
-		(property "LCSC" "C7303451"
+		(property "LCSC" "C603545"
 			(at 180.34 58.42 0)
 			(effects

Commit message: fix(pcb): resize Y1 crystal load caps to 30pF to match 18pF spec
Update crystal load capacitors C6 and C9 from 27pF to 30pF (0402CG300J500NT, LCSC C1570) across the schematic, PCB layout, and JLCPCB manufacturing BOM.

With series capacitance C_series = (30 * 30)/(30 + 30) = 15.0 pF and typical 6-layer stray capacitance C_stray ≈ 2.5–3.0 pF, this yields an effective load capacitance of 17.5–18.0 pF, reconciling the previous documentation discrepancy where 27pF caps yielded only 16.0 pF against the 18pF nominal specification of Y1 (ECS-192-18-33-JGN-TR). Update READMEs and validation documentation accordingly.

Co-Authored-By: CopperPilot <noreply@copperpilot.ai>
Parts:
- C6, C9: value 27p -> 30p; LCSC C1557 -> C1570; MPN 0402CG270J500NT -> 0402CG300J500NT
Changed lines of the file:
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@@
 			)
 		)
-		(property "Value" "27p"
+		(property "Value" "30p"
 			(at 109.22 155.956 90)
 			(hide yes)
@@
 			)
 		)
-		(property "Description" "18pF 50V C0G 0402 MLCC"
+		(property "Description" "30pF 50V C0G 0402 MLCC"
 			(at 109.22 149.86 0)
 			(hide yes)
@@
 			)
 		)
-		(property "MPN" "0402CG270J500NT"
+		(property "MPN" "0402CG300J500NT"
 			(at 109.22 149.86 0)
 			(effects
@@
 			)
 		)
-		(property "LCSC" "C1557"
+		(property "LCSC" "C1570"
 			(at 109.22 149.86 0)
 			(effects
@@
 			)
 		)
-		(property "Value" "27p"
+		(property "Value" "30p"
 			(at 109.22 176.276 90)
 			(hide yes)
@@
 			)
 		)
-		(property "Description" "18pF 50V C0G 0402 MLCC"
+		(property "Description" "30pF 50V C0G 0402 MLCC"
 			(at 109.22 170.18 0)
 			(hide yes)
@@
 			)
 		)
-		(property "MPN" "0402CG270J500NT"
+		(property "MPN" "0402CG300J500NT"
 			(at 109.22 170.18 0)
 			(effects
@@
 			)
 		)
-		(property "LCSC" "C1557"
+		(property "LCSC" "C1570"
 			(at 109.22 170.18 0)
 			(effects
