File: pcb/rp3a0-mini.kicad_pcb (KiCad board)
At the start: 6 copper layers, 60 x 20.4 mm, 124 parts, among them J1 473092651, J2 467652301, J3 1054500101, J4 SOLDER_PAD_OPEN, J5 PICO_PADS, Q1 DMG2305UX-7, U1 RP3A0-AU, U2 RT9081A-1BGQZA(2), U3 RT8088AWSC, U4 PAM2306AYPKE, U5 DMN2004VK-7, Y1 19.2MHz

Commit message: fix(pcb): update 19.2MHz crystal load caps to 27pF, add PCB title block, and export JLCPCB BOM/CPL
Update C6 and C9 from 18pF to 27pF (0402CG270J500NT, LCSC C1557) to provide 18.0 pF effective load capacitance for Y1 (ECS-192-18-33-JGN-TR), add PCB title_block metadata, and configure export_manufacturing.py with JLCPCB_CORRECTIONS and tracked pcb/jlcpcb/ BOM/CPL outputs.

Co-Authored-By: CopperPilot <noreply@copperpilot.ai>
Parts:
- C6, C9: value 18p -> 27p
Changed lines of the file:
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@@
 	)
 	(paper "A4")
+	(title_block
+		(title "RP3A0 Pico")
+		(date "2026-03-06")
+		(rev "1.1")
+		(comment 1 "Raspberry Pi Zero 2W RP3A0-AU SiP in Pi Pico Form Factor")
+		(comment 2 "6-Layer PCB for JLCPCB Manufacturing")
+	)
 	(layers
 		(0 "F.Cu" signal "Top Layer")
@@
 			)
 		)
-		(property "Value" "18p"
+		(property "Value" "27p"
 			(at -5.398155 7.432802 0)
 			(unlocked yes)
@@
 			)
 		)
-		(property "MPN" "0402CG180J500NT"
+		(property "MPN" "0402CG270J500NT"
 			(at 159.0011 100.6286 0)
 			(layer "F.Fab")
@@
 			)
 		)
-		(property "LCSC" "C1549"
+		(property "LCSC" "C1557"
 			(at 159.0011 100.6286 0)
 			(layer "F.Fab")
@@
 			)
 		)
-		(property "Value" "18p"
+		(property "Value" "27p"
 			(at 2.475845 2.098802 0)
 			(unlocked yes)
@@
 			)
 		)
-		(property "MPN" "0402CG180J500NT"
+		(property "MPN" "0402CG270J500NT"
 			(at 159.0011 99.7286 0)
 			(layer "F.Fab")
@@
 			)
 		)
-		(property "LCSC" "C1549"
+		(property "LCSC" "C1557"
 			(at 159.0011 99.7286 0)
 			(layer "F.Fab")

Commit message: fix(pcb): resolve S2/S6/S7 validation findings across BOM, footprints, and 6-layer PCB
- Swap D1 (KT-0603G, C12624) symbol and PCB pad polarity so Pin 1 (K) connects to STATUS_LED and Pin 2 (A) to 3V3 via R11
- Replace U2 adjustable LCSC code with fixed 1.25V 500mA VBIAS LDO NCP133AMX125TCG (C603545) matching pinout and footprint
- Upgrade Y1 (S3219200182080C3, C5380596), U5 (DMN601VK-7, C110498), and R12/R13/R18 (RC0402FR-07240RL, C114755) to stocked JLCPCB parts
- Expand C0805_NP (C12, C14) inner pad gap to 0.70 mm and set 0 mm solder mask margin on fine-pitch U3 and J2
- Add D2 cathode bar, F.Fab/F.CrtYd outlines across all footprints, 3 global optical fiducials (FID1-FID3), and In4.Cu GND reference pour

Co-Authored-By: CopperPilot <noreply@copperpilot.ai>
Parts:
- U2: value RT9081A-1BGQZA(2) -> NCP133AMX125TCG
- U5: value DMN2004VK-7 -> DMN601VK-7
- turned D1 to 90 degrees
Connections:
- D1 pad 1: Net-(D1-Pad1) -> Net-(U1G-STATUS_LED)
- D1 pad 2: Net-(U1G-STATUS_LED) -> Net-(D1-Pad2)
- R11 pad 2: Net-(D1-Pad1) -> Net-(D1-Pad2)
Routing:
- net Net-(D1-Pad2): track 0.00 -> 1.12 mm
- net Net-(D1-Pad1): track 1.12 -> 0.00 mm
- added copper zone on In4.Cu, net GND
Other:
- board text added: "FID1"
- board text added: "FID2"
- board text added: "FID3"

Commit message: fix(pcb): resize Y1 crystal load caps to 30pF to match 18pF spec
Update crystal load capacitors C6 and C9 from 27pF to 30pF (0402CG300J500NT, LCSC C1570) across the schematic, PCB layout, and JLCPCB manufacturing BOM.

With series capacitance C_series = (30 * 30)/(30 + 30) = 15.0 pF and typical 6-layer stray capacitance C_stray ≈ 2.5–3.0 pF, this yields an effective load capacitance of 17.5–18.0 pF, reconciling the previous documentation discrepancy where 27pF caps yielded only 16.0 pF against the 18pF nominal specification of Y1 (ECS-192-18-33-JGN-TR). Update READMEs and validation documentation accordingly.

Co-Authored-By: CopperPilot <noreply@copperpilot.ai>
Parts:
- C6, C9: value 27p -> 30p
Changed lines of the file:
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@@
 			)
 		)
-		(property "Value" "27p"
+		(property "Value" "30p"
 			(at -5.398155 7.432802 0)
 			(unlocked yes)
@@
 			)
 		)
-		(property "Description" "18pF 50V C0G 0402 MLCC"
+		(property "Description" "30pF 50V C0G 0402 MLCC"
 			(at 0 0 0)
 			(layer "F.Fab")
@@
 			)
 		)
-		(property "MPN" "0402CG270J500NT"
+		(property "MPN" "0402CG300J500NT"
 			(at 159.0011 100.6286 0)
 			(layer "F.Fab")
@@
 			)
 		)
-		(property "LCSC" "C1557"
+		(property "LCSC" "C1570"
 			(at 159.0011 100.6286 0)
 			(layer "F.Fab")
@@
 			)
 		)
-		(property "Value" "27p"
+		(property "Value" "30p"
 			(at 2.475845 2.098802 0)
 			(unlocked yes)
@@
 			)
 		)
-		(property "Description" "18pF 50V C0G 0402 MLCC"
+		(property "Description" "30pF 50V C0G 0402 MLCC"
 			(at 0 0 0)
 			(layer "F.Fab")
@@
 			)
 		)
-		(property "MPN" "0402CG270J500NT"
+		(property "MPN" "0402CG300J500NT"
 			(at 159.0011 99.7286 0)
 			(layer "F.Fab")
@@
 			)
 		)
-		(property "LCSC" "C1557"
+		(property "LCSC" "C1570"
 			(at 159.0011 99.7286 0)
 			(layer "F.Fab")
